File: BMS.kicad_pcb (KiCad board)
At the start: 4 copper layers, 121.9 x 78.7 mm, 108 parts, among them J1 Conn_02x02_Counter_Clockwise, J10 OLED, J2 Conn_02x02_Counter_Clockwise, J3 RJ45, J4 Conn_02x08_Top_Bottom, J5 Conn_02x05_Top_Bottom, J6 Conn_02x02_Counter_Clockwise, Q2 SIRA00DP-T1-GE3, Q5 Q_NMOS, Q6 Q_NMOS, Q7 Q_NMOS, Q8 Q_NMOS, SW1 SW_DIP_x01, SW2 SW_DIP_x01, SW3 SW_DIP_x01, U1 K7805M-1000R3, U10 TJA1051T/3/1J, U11 TPS2051CDBV, U12 TPS2051CDBV, U13 TPS2051CDBV, U14 CA-IS3740, U16 DGD0211CWT-7, U17 DGD0211CWT-7, U18 DGD0211CWT-7, U19 DGD0211CWT-7, U2 B0505S-3WR2, U3 Teensy4.1, U4 VND7050AJTR, U5 TJA1051T/3/1J, U6 ISO7331C, U7 TPS2051CDBV, U8 VND7050AJTR, U9 ISO1050DWR

Commit message: Added 12v Out Protection, generally completed layout
Parts:
- removed C15, C16: 1uF, Capacitor_SMD:C_0603_1608Metric
- removed Q5, Q6, Q7, Q8: Q_NMOS, Package_SO:SOP-8_3.9x4.9mm_P1.27mm
- removed U17, U18, U19: DGD0211CWT-7, Package_TO_SOT_SMD:SOT-23-5
- added D30: D, Diode_SMD:D_0805_2012Metric, F.Cu at (83.7, 101.4)
- added R41: 1k, Resistor_SMD:R_0603_1608Metric, F.Cu at (108.7, 100.7)
- added R42: 1k, Resistor_SMD:R_0603_1608Metric, F.Cu at (109.6, 103.7)
- added R43: 1k, Resistor_SMD:R_0603_1608Metric, F.Cu at (110.8, 100.7)
- added R44: 1k, Resistor_SMD:R_0603_1608Metric, F.Cu at (111.8, 103.7)
- added R45: 1k, Resistor_SMD:R_0603_1608Metric, F.Cu at (112.8, 100.7)
- added R46: 1k, Resistor_SMD:R_0603_1608Metric, F.Cu at (114.0, 103.7)
- added R47: 1k, Resistor_SMD:R_0603_1608Metric, F.Cu at (115.0, 100.7)
- added R48: 1k, Resistor_SMD:R_0603_1608Metric, F.Cu at (116.2, 103.7)
- added R49: 47k, Resistor_SMD:R_0603_1608Metric, F.Cu at (118.5, 103.5)
- added R50: 47k, Resistor_SMD:R_0603_1608Metric, F.Cu at (118.5, 101.9)
- added R51: 47k, Resistor_SMD:R_0603_1608Metric, F.Cu at (106.2, 102.0)
- added R52: 47k, Resistor_SMD:R_0603_1608Metric, F.Cu at (106.2, 103.5)
- added U15: VNLD5090TR-E, Package_SO:SO-8_3.9x4.9mm_P1.27mm, F.Cu at (108.8, 94.5)
- added U20: VNLD5090TR-E, Package_SO:SO-8_3.9x4.9mm_P1.27mm, F.Cu at (115.4, 94.5)
- C13: value 1uF -> 470uF; footprint Capacitor_SMD:C_0603_1608Metric -> Capacitor_SMD:CP_Elec_10x10
- R37: value 8 -> 4.7k
- R38, R39: value 8 -> 15k
- R40: value 8 -> 1k
- TP1, TP4: footprint TestPoint:TestPoint_Pad_2.5x2.5mm -> user:Clip_TP
- TP2, TP3, TP5, TP6: footprint TestPoint:TestPoint_Pad_2.5x2.5mm -> user:STD_TP
- U16: value DGD0211CWT-7 -> VND7050AJTR; footprint Package_TO_SOT_SMD:SOT-23-5 -> Package_SO:PowerSSO-16-1EP_3.9x4.9mm_P0.5mm_EP2.5x3.61mm_ThermalVias
- moved TP4 186.8 mm to (81.0, 112.2), turned to 90 degrees
- moved TP6 184.0 mm to (80.9, 121.3)
- moved TP5 179.9 mm to (80.9, 128.6)
- moved TP2 177.6 mm to (80.7, 83.5)
- moved C14 80.5 mm to (141.6, 132.0), turned to 180 degrees
- moved C13 77.2 mm to (148.5, 141.8)
- moved D6 63.9 mm to (97.7, 99.4), turned to 90 degrees
- moved D16 62.9 mm to (102.9, 103.3), turned to 90 degrees
- moved D9 60.7 mm to (95.9, 103.3), turned to 90 degrees
- moved D15 59.2 mm to (99.4, 103.3), turned to 90 degrees
- moved D8 57.8 mm to (92.4, 103.3), turned to 90 degrees
- moved R16 53.5 mm to (102.9, 99.4), turned to 90 degrees
- moved R15 50.2 mm to (99.4, 99.4), turned to 90 degrees
- moved R13 48.6 mm to (97.6, 96.1), turned to 90 degrees
- moved U16 46.7 mm to (85.3, 93.6), turned to 90 degrees
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Connections:
- C13 pad 1: GND -> /Overcurrent_Protection3/V_{OUT}
- C13 pad 2: +5V -> GND_ISO
- C14 pad 1: GND -> /Overcurrent_Protection3/V_{OUT}
- C14 pad 2: +5V -> GND_ISO
- J4 pad 10: +12V -> /12V_Out_Bank2
- J4 pad 11: +12V -> /12V_Out_Bank2
- J4 pad 9: +12V -> /12V_Out_Bank1
- R37 pad 1: Net-(U19-OUT) -> /12V_Output_Protection/Driver_Gnd
- R37 pad 2: Net-(Q5-G) -> GND
- R38 pad 1: Net-(U16-OUT) -> +5V
- R38 pad 2: Net-(Q6-G) -> Net-(U16-Input_0)
- R39 pad 1: Net-(U17-OUT) -> +5V
- R39 pad 2: Net-(Q7-G) -> Net-(U16-Input_1)
- R40 pad 1: Net-(U18-OUT) -> GND
- R40 pad 2: Net-(Q8-G) -> Net-(U16-Multisense)
- U16 pad 1: +5V -> Net-(U16-Input_0)
- U16 pad 3: /OUT6_LSD_LOGIC -> unconnected-(U16-SEn-Pad3)
- U16 pad 4: GND -> /12V_Output_Protection/Driver_Gnd
- U16 pad 5: Net-(U16-OUT) -> unconnected-(U16-Select_0-Pad5)
- U3 pad 17: unconnected-(U3-25_A11_RX6_SDA2-Pad17) -> /OUT5_LSD_Status
- U3 pad 18: unconnected-(U3-26_A12_MOSI1-Pad18) -> /OUT6_LSD_Status
- U3 pad 19: unconnected-(U3-27_A13_SCK1-Pad19) -> /OUT7_LSD_Status
- U3 pad 20: unconnected-(U3-28_RX7-Pad20) -> /OUT8_LSD_Status
- U3 pad 38: unconnected-(U3-16_A2_RX4_SCL1-Pad38) -> /Logic_IN_1
- U3 pad 39: unconnected-(U3-17_A3_TX4_SDA1-Pad39) -> /Logic_IN_2
- U3 pad 40: unconnected-(U3-18_A4_SDA-Pad40) -> /Logic_IN_3
- U3 pad 41: unconnected-(U3-19_A5_SCL-Pad41) -> /Logic_IN_4
Routing:
- net /OUT4_HSD_LOGIC: track 0.00 -> 98.1 mm, vias 0 -> 1
- net /OUT5_LSD_LOGIC: track 0.00 -> 94.3 mm, vias 0 -> 1
- net /OUT3_HSD_LOGIC: track 0.00 -> 90.4 mm, vias 0 -> 1
- net /OUT2_HSD_LOGIC: track 0.00 -> 90.2 mm, vias 0 -> 1
- net /OUT1_HSD_LOGIC: track 0.00 -> 88.7 mm, vias 0 -> 1
- net /OUT6_LSD_LOGIC: track 0.00 -> 88.5 mm, vias 0 -> 1
- net /CAN1_TX: track 0.00 -> 81.9 mm, vias 0 -> 3
- net /CAN1_RX: track 0.00 -> 80.5 mm, vias 0 -> 3
- net /OUT7_LSD_LOGIC: track 0.00 -> 79.9 mm, vias 0 -> 1
- net /OUT8_LSD_LOGIC: track 0.00 -> 74.3 mm, vias 0 -> 1
- net /RTC_BATT_+: track 0.00 -> 71.3 mm, vias 0 -> 2
- net /CAN3_RX: track 0.00 -> 57.6 mm, vias 0 -> 2
- net /SERIAL_RX: track 0.00 -> 56.5 mm, vias 0 -> 2
- net /OUT5_LSD_Status: track 0.00 -> 56.4 mm, vias 0 -> 1
- net /SERIAL_TX: track 0.00 -> 55.7 mm, vias 0 -> 2
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- added copper zone on F.Cu, net /12V_Out_Bank1
- added copper zone on In1.Cu, net /12V_Out_Bank1
- added copper zone on B.Cu, net /12V_Out_Bank2
- added copper zone on F.Cu, net /12V_Out_Bank2
- added copper zone on In2.Cu, net /12V_Out_Bank2
- added copper zone on F.Cu, net /OUT5_LSD_PWR
- added copper zone on In1.Cu, net /OUT5_LSD_PWR
- added copper zone on B.Cu, net /OUT6_LSD_PWR
- added copper zone on F.Cu, net /OUT6_LSD_PWR
- added copper zone on In2.Cu, net /OUT6_LSD_PWR
- added copper zone on F.Cu, net /OUT7_LSD_PWR
- added copper zone on In1.Cu, net /OUT7_LSD_PWR
- added copper zone on B.Cu, net /OUT8_LSD_PWR
- added copper zone on F.Cu, net /OUT8_LSD_PWR
- added copper zone on In2.Cu, net /OUT8_LSD_PWR
- added copper zone on In1.Cu, net GND
- added copper zone on In2.Cu, net GND
Other:
- board text added: "!FUSE"
- board text added: "12V"
- board text added: "12V_{IN} GND_{IN}"
- board text added: "3.3V"
- board text added: "5V"
- board text added: "5V_ISO"
- board text added: "GND"
- board text added: "GND_ISO"
- board text added: "H2 H4 H1 H3"
- board text added: "J4 POWER CONN"
- board text added: "L6 L8 L5 L7"
- board text added: "Teensy 4.1"
- board text added: "USB"

Commit message: All the diodes, and other layout work
Parts:
- added D31: D, Diode_SMD:D_SOD-123, F.Cu at (158.4, 84.3)
- added D32: D, Diode_SMD:D_SOD-123, F.Cu at (162.3, 85.9)
- added D33: BAT54S, Package_TO_SOT_SMD:SOT-523, F.Cu at (107.3, 113.7)
- added D34: BAT54S, Package_TO_SOT_SMD:SOT-523, F.Cu at (109.5, 113.7)
- added D35: BAT54S, Package_TO_SOT_SMD:SOT-523, F.Cu at (111.8, 115.2)
- added D36: BAT54S, Package_TO_SOT_SMD:SOT-523, F.Cu at (114.0, 115.2)
- added D37: BAT54S, Package_TO_SOT_SMD:SOT-523, F.Cu at (119.4, 96.9)
- added D38: BAT54S, Package_TO_SOT_SMD:SOT-523, F.Cu at (116.3, 115.2)
- added D39: BAT54S, Package_TO_SOT_SMD:SOT-523, F.Cu at (121.7, 96.9)
- added D40: BAT54S, Package_TO_SOT_SMD:SOT-523, F.Cu at (118.6, 115.2)
- added Q1: BSS138LT1G, Package_TO_SOT_SMD:SOT-23, F.Cu at (159.2, 87.7)
- added R53: 4.7k, Resistor_SMD:R_0603_1608Metric, F.Cu at (159.0, 90.9)
- added R54: 330, Resistor_SMD:R_0603_1608Metric, F.Cu at (162.6, 90.9)
- D15, D16, D8, D9: footprint Package_TO_SOT_SMD:SOT-23 -> Package_TO_SOT_SMD:SOT-523
- D30, D6: footprint Diode_SMD:D_0805_2012Metric -> Diode_SMD:D_SOD-123
- Q2: value SIRA00DP-T1-GE3 -> HSBA100P03
- moved SW1 9.99 mm to (114.6, 131.6), turned to 180 degrees
- moved R31 4.72 mm to (80.0, 74.9)
- moved D24 3.25 mm to (86.1, 71.4), turned to 180 degrees
- moved R5 3.00 mm to (106.4, 115.8)
- moved R4 2.96 mm to (106.4, 117.3)
- moved U11 2.84 mm to (80.3, 78.0), turned to 180 degrees
- moved R1 1.55 mm to (122.7, 74.2)
- moved D1 1.52 mm to (126.5, 74.2)
- moved R2 1.26 mm to (118.6, 129.3)
- moved D8 0.32 mm to (92.4, 103.0)
- moved D9 0.31 mm to (95.9, 103.0)
- moved D15 0.31 mm to (99.4, 103.0)
- moved D16 0.31 mm to (102.9, 103.0)
- turned D30 to -90 degrees
Connections:
- C1 pad 1: Net-(BZ1--) -> Net-(D1-K)
- D1 pad 1: Net-(BZ1--) -> Net-(D1-K)
- F1 pad 2: Net-(BZ1--) -> Net-(D1-K)
- L1 pad 1: Net-(BZ1--) -> Net-(D1-K)
- U3 pad 12: unconnected-(U3-10_CS_MQSR-Pad12) -> /Buzzer_Logic
- U3 pad 16: V_Supply_Sense -> I2C_SCL
- U3 pad 17: /OUT5_LSD_Status -> I2C_SDA
- U3 pad 18: /OUT6_LSD_Status -> /OUT5_LSD_Status
- U3 pad 19: /OUT7_LSD_Status -> /OUT6_LSD_Status
- U3 pad 20: /OUT8_LSD_Status -> /OUT7_LSD_Status
- U3 pad 21: unconnected-(U3-29_TX7-Pad21) -> /OUT8_LSD_Status
Routing:
- net Net-(BZ1--): track 48.5 -> 8.69 mm, vias 1 -> 0
- net I2C_SDA: track 0.00 -> 27.0 mm, vias 0 -> 1
- net I2C_SCL: track 0.00 -> 25.2 mm
- net GND: track 21.0 -> 39.1 mm, vias 41 -> 49
- net +3.3V: track 33.9 -> 51.3 mm, vias 10 -> 13
- net Net-(D1-K): track 0.00 -> 10.0 mm, vias 0 -> 1
- net /OUT6_LSD_Status: track 50.4 -> 59.9 mm, vias 1 -> 3
- net /OUT8_LSD_LOGIC: track 74.3 -> 83.6 mm, vias 1 -> 3
- net /OUT7_LSD_LOGIC: track 79.9 -> 88.4 mm, vias 1 -> 3
- net /OUT6_LSD_LOGIC: track 88.5 -> 96.8 mm, vias 1 -> 3
- net /OUT7_LSD_Status: track 42.7 -> 50.9 mm, vias 3 -> 5
- net /OUT8_LSD_Status: track 36.3 -> 44.3 mm, vias 1 -> 3
- net /OUT5_LSD_LOGIC: track 94.3 -> 102.0 mm, vias 1 -> 3
- net /OUT5_LSD_Status: track 56.4 -> 63.6 mm, vias 1 -> 3
- net /CAN1_HIGH_ISO: track 29.3 -> 23.2 mm
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- added copper zone on F.Cu, net Net-(D1-K)
- removed copper zone on F.Cu, net Net-(BZ1--)
Other:
- board text added: "5V TX GND RX"
- board text added: "C_{1}H"
- board text added: "C_{1}L"
- board text added: "J1 - UART"
- board text added: "J2 - CURRENT"
- board text added: "J3 - CAN3 RJ45"
- board text added: "J4 - POWER"
- board text added: "J5 - AUX COMMS"
- board text added: "J6 - CAN1"
- board text added: "PLEASE MIND THE (ISOLATION) GAP"
- board text added: "TR120"
- board text removed: "J4 POWER CONN"
