File: BMS.kicad_sch (KiCad schematic)
At the start: 56 parts, among them J1 Conn_02x02_Counter_Clockwise, J10 OLED, J2 Conn_02x02_Counter_Clockwise, J3 RJ45, J4 Conn_02x08_Top_Bottom, J5 Conn_02x05_Top_Bottom, J6 Conn_02x02_Counter_Clockwise, J7 Conn_02x02_Counter_Clockwise, Q1 BSS138LT1G, Q2 HSBA100P03, Q3 BSS138LT1G, Q4 BSS138LT1G, U1 K7805M-1000R3, U14 CA-IS3740, U2 B0505S-3WR2, U3 Teensy4.1

Commit message: Schematic Layout Improvements, Start of RS485 Circuit
Parts:
- added C15: 1uF, Capacitor_SMD:C_0603_1608Metric, symbol Device:C
- added U18: SN65HVD11HD, Package_SO:SOIC-8_3.9x4.9mm_P1.27mm, symbol Interface_UART:SN65HVD11HD
Connections:
- net +3.3V: now also C15.2, U18.8 (VCC)
- net GND: now also C15.1, U18.5 (GND)
- new net RS485_BUS_A: U18.6 (A)
- new net RS485_BUS_B: U18.7 (B)
Other:
- note added: "CAN Connector ISOLATED"
- note added: "Connector J2 - Analogue Current"
- note added: "Connector J3 - RJ45 CAN3"
- note added: "Connector J4 - POWER"
- note added: "Connector J5 - Auxillary Comms"
- note added: "Connector J7 - RS485/Modbus"
- note added: "Isolated Circuits"
- note added: "Isolated Power Supply"
- note added: "Serial Connector ISOLATED"
- note added: "Teensy 4.1"
- note removed: "Teensy"
- moved on the sheet: BT1, BZ1, C1, C11, C12, C13, C14, C2, D1, D21, D22, D27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

Commit message: Finalised RS485 Circuit, Layout improvemnts, mounting holes, silkscreen...
Parts:
- added BC1, BC2: Conn_01x24, eChook:BC, symbol Connector_Generic:Conn_01x24
- added BC3: Conn_01x02, eChook:BC, symbol Connector_Generic:Conn_01x02
- added C16, C17: 4.7uF, Capacitor_SMD:C_0603_1608Metric, symbol Device:C
- added C18: 470uF, Capacitor_SMD:CP_Elec_10x10, symbol Device:C_Polarized
- added D43: SM712_SOT23, Package_TO_SOT_SMD:SOT-23, symbol Diode:SM712_SOT23
- added D44, D45: BAT54S, Package_TO_SOT_SMD:SOT-523, symbol Diode:BAT54S
- added H1, H2, H3, H4: MountingHole, MountingHole:MountingHole_3.2mm_M3_Pad_TopBottom, symbol Mechanical:MountingHole
- added J8: Conn_02x08_Top_Bottom, Connector_PinHeader_1.27mm:PinHeader_2x08_P1.27mm_Vertical_SMD, symbol Connector_Generic:Conn_02x08_Odd_Even
- added JP1, JP2: SolderJumper_3_Bridged12, Jumper:SolderJumper-3_P1.3mm_Bridged12_RoundedPad1.0x1.5mm, symbol Jumper:SolderJumper_3_Bridged12
- added R61, R62: 10, Resistor_SMD:R_1206_3216Metric, symbol Device:R
- added R63, R64: 10k, Resistor_SMD:R_0603_1608Metric, symbol Device:R
- added R65, R66, R67, R68, R69, R70: 3.3k, Resistor_SMD:R_0402_1005Metric, symbol Device:R
- BT1: LCSC (none) -> C18212226
- D42: footprint LED_SMD:LED_0603_1608Metric -> LED_SMD:LED_0805_2012Metric; LCSC (none) -> C2297
- J3: LCSC (none) -> C708654
- R1, R28: footprint Resistor_SMD:R_0805_2012Metric -> Resistor_SMD:R_0603_1608Metric; LCSC C17414 -> (none)
- TP1, TP2, TP3, TP4, TP5, TP6, U3: now left out of the parts list
Connections:
- net +12V: now also C18.1, J8.3 (Pin_3), J8.4 (Pin_4), J8.7 (Pin_7), J8.8 (Pin_8)
- net +3.3V: now also U14.10 (EN_{B}), D44.2 (K), D45.2 (K), R63.2
- net +5V: now also U14.7 (EN_{A})
- net CAN2_RX: now also JP2.1 (A), JP2.2 (C)
- net CAN2_TX: now also JP1.1 (A), JP1.2 (C)
- net CAN3_HIGH: now also J8.13 (Pin_13), J8.14 (Pin_14)
- net CAN3_LOW: now also J8.15 (Pin_15), J8.16 (Pin_16)
- net Current_Sense_In_High: now also R68.1
- net Current_Sense_In_Low: now also R65.1
- net GND: now also J7.1 (Pin_1), J7.2 (Pin_2), C16.2, C17.2, C18.2, D43.3 (common), D44.1 (A), D45.1 (A), J8.1 (Pin_1), J8.10 (Pin_10), J8.2 (Pin_2), J8.9 (Pin_9), R64.1, R67.2, R70.2; no longer U14.10 (EN_{B}), U14.7 (EN_{A})
- net RS485_BUS_A: now also J7.3 (Pin_3), D43.2 (A2), R62.2; no longer U18.6 (A)
- net RS485_BUS_B: now also J7.4 (Pin_4), D43.1 (A1), R61.2; no longer U18.7 (B)
- net RS-485_DIR: now reaches U3.11 (9_OUT1C)
- net RS-485_DIR: now also U18.2 (~{RE}), U18.3 (DE), R64.2
- net Curr_Sens_High_3v3: now reaches U3.36 (14_A0_TX3_SPDIF_OUT)
- net Curr_Sens_High_3v3: now also C17.1, D45.3 (COM), R68.2, R69.1
- net Curr_Sens_Low_3v3: now reaches U3.37 (15_A1_RX3_SPDIF_IN)
- net Curr_Sens_Low_3v3: now also C16.1, D44.3 (COM), R65.2, R66.1
- net at J3.3: now also J8.5 (Pin_5)
- net at J3.6: now also J8.11 (Pin_11)
- net RS-485_Rx: now reaches U18.1 (R)
- net RS-485_Rx: now also JP2.3 (B), R63.1
- net RS-485_Tx: now reaches U18.4 (D)
- net RS-485_Tx: now also JP1.3 (B)
- new net: R62.1, U18.6 (A)
- new net: R66.2, R67.1
- new net: R69.2, R70.1
- new net: R61.1, U18.7 (B)
Other:
- note added: "9.4Hz LPF"
- note added: "BOM Placeholders"
- note added: "CAN2/RS-485 Switch"
- note added: "Current Input Voltage Divider"
- note added: "Hardware License"
- note added: "Mounting Holes"
- note added: "No footprint items to hold part numbers for Teensy Headers"
- note added: "RS-485 Interface"
- note added: "TODO - check U14 Footprint. JLC Render is tiny SSOP16"
- note added: "eChook Non-Commercial Open Hardware License (Version 1.0) Copyright (c) 2025 eChook 1. License Grant Permission is hereby granted, free of charge, to any person obtaining a copy of this hardware design and associated documentation (the "Design"), to use, modify, and distribute the Design, subject to the following conditions: 2. Non-Commercial Use Only This Design may not be used for commercial pu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"
- company: (none) -> eChook
- title: (none) -> BMS Comms Master Board
- moved on the sheet: J3

Commit message: Pinout swapped for PWMable Error LED
Connections:
- net ERROR_LED: now also U3.25 (33_MCLK2); no longer U3.24 (32_OUT1B)
- net HSD_SEL_0_A: now also U3.24 (32_OUT1B); no longer U3.25 (33_MCLK2)
Other:
- note added: "TODO - RX/TX2 Aren't connected and we're out of pins!"
Changed lines of the file:
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@@
 		)
 	)
+	(text "TODO - RX/TX2 Aren't connected and we're out of pins!"
+		(exclude_from_sim no)
+		(at 480.822 320.294 0)
+		(effects
+			(font
+				(size 1.27 1.27)
+			)
+		)
+	)
 	(text "Active LEDs"
 		(exclude_from_sim no)
@@
 	)
 	(label "ERROR_LED"
-		(at 166.37 168.91 180)
+		(at 69.85 168.91 0)
 		(effects
 			(font
 				(size 1.27 1.27)
 			)
-			(justify right bottom)
+			(justify left bottom)
 		)
 	)
@@
 	)
 	(label "HSD_SEL_0_A"
-		(at 69.85 168.91 0)
+		(at 166.37 168.91 180)
 		(effects
 			(font
 				(size 1.27 1.27)
 			)
-			(justify left bottom)
+			(justify right bottom)
 		)
 	)

Commit message: Added UART Buffer for Aux Connector Serial
Parts:
- added R71, R72: 4.7k, Resistor_SMD:R_0603_1608Metric, symbol Device:R
Connections:
- net +3.3V: now also R71.2, R72.2
- net I2C_SCL: now also R71.1
- net I2C_SDA: now also R72.1
- net CAN2_HIGH renamed CAN2_HIGH_Ext
- net CAN2_LOW renamed CAN2_LOW_Ext
- net CAN3_HIGH renamed CAN3_HIGH_Ext
- net CAN3_LOW renamed CAN3_LOW_Ext
- net In_1 renamed In_1_Ext
- net In_2 renamed In_2_Ext
- net In_3 renamed In_3_Ext
- net In_4 renamed In_4_Ext
- net OUT5_LSD_Status: no longer names the net of U3.18 (26_A12_MOSI1)
- net OUT6_LSD_Status: no longer names the net of U3.19 (27_A13_SCK1)
- net OUT7_LSD_Status renamed RX_2_logic
- net OUT8_LSD_Status renamed TX_2_logic
- net RX_2 renamed RX_2_Ext
- net TX_2 renamed TX_2_Ext
- no-connect marks 0 -> 54
Other:
- added sheet Isolated_UART1 (UART_Isolated_Interface.kicad_sch)
- note added: "UART Buffer"
- note removed: "TODO - RX/TX2 Aren't connected and we're out of pins!"
- moved on the sheet: J10, J3, J7, J8

Commit message: Added hieracical schematic for better 5V_OUT protection
Other:
- added sheet 5V_OUT_PROT (5V_OCP_OVP_RPP.kicad_sch)
- note added: "TODO: Free up some serial pins do CAN3 and RS485 don't have to share"
- note added: "TODO: Multisense signals need to go to Analogue INputs!"
Changed lines of the file:
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@@
 		)
 	)
+	(text "TODO: Multisense signals need to go to Analogue INputs!"
+		(exclude_from_sim no)
+		(at 74.676 148.844 0)
+		(effects
+			(font
+				(size 1.27 1.27)
+			)
+		)
+	)
 	(text "CAN Transceivers - Non Isolated"
 		(exclude_from_sim no)
@@
 		)
 	)
+	(text "TODO: Free up some serial pins do CAN3 and RS485 don't have to share"
+		(exclude_from_sim no)
+		(at 79.756 154.94 0)
+		(effects
+			(font
+				(size 1.27 1.27)
+			)
+		)
+	)
 	(text "Serial Connector ISOLATED"
 		(exclude_from_sim no)
@@
 				)
 			)
+		)
+	)
+	(sheet
+		(at 469.265 290.195)
+		(size 26.67 11.43)
+		(exclude_from_sim yes)
+		(in_bom no)
+		(on_board no)
+		(dnp yes)
+		(fields_autoplaced yes)
+		(stroke
+			(width 0.1524)
+			(type solid)
+		)
+		(fill
+			(color 0 0 0 0.0000)
+		)
+		(property "Sheetname" "5V_OUT_PROT"
+			(at 469.265 289.4834 0)
+			(effects
+				(font
+					(size 1.27 1.27)
+				)
+				(justify left bottom)
+			)
+		)
+		(property "Sheetfile" "5V_OCP_OVP_RPP.kicad_sch"
+			(at 469.265 302.2096 0)
+			(effects
+				(font
+					(size 1.27 1.27)
+				)
+				(justify left top)
+			)
+		)
+		(property "Field2" ""
+			(at 469.265 290.195 0)
+			(effects
+				(font
+					(size 1.27 1.27)
+				)
+			)
+		)
+		(instances
+			(project "BMS"
+				(path "/d7e219ab-f530-45f5-8a23-0e6b6d2e3e0f"
+					(page "14")
+				)
+			)

Commit message: Fixed network pinouts - no shared pins now
Parts:
- removed JP2: SolderJumper_3_Bridged12, Jumper:SolderJumper-3_P1.3mm_Bridged12_RoundedPad1.0x1.5mm, symbol Jumper:SolderJumper_3_Bridged12
- removed U3: Teensy4.1, teensy_library:Teensy_4.1_RTC, symbol teensy:Teensy4.1
- added C25: 10uF, Capacitor_SMD:C_0805_2012Metric, symbol Device:C
- added C26: 22uF, Capacitor_SMD:C_0603_1608Metric, symbol Device:C
- added C27: 10uF, Capacitor_SMD:C_0603_1608Metric, symbol Device:C
- added C28: 4.7uF, Capacitor_SMD:C_0603_1608Metric, symbol Device:C
- added U3: Teensy4.1, teensy_library:Teensy_4.1_RTC, symbol user:Teensy4.1
- BC1, BC2: symbol Connector_Generic:Conn_01x24 -> Mechanical:MountingHole
- BC3: symbol Connector_Generic:Conn_01x02 -> Mechanical:MountingHole
- H1, H2, H3, H4: footprint MountingHole:MountingHole_3.2mm_M3_Pad_TopBottom -> MountingHole:MountingHole_3.2mm_M3_Pad; symbol Mechanical:MountingHole -> Mechanical:MountingHole_Pad
- U14: footprint Package_SO:SOIC-16W_7.5x10.3mm_P1.27mm -> Package_SO:SSOP-16_3.9x4.9mm_P0.635mm
Connections:
- net +12V: now also C25.2; no longer Q2.6 (D), Q2.7 (D), Q2.8 (D)
- net +3.3V: now also JP1.3 (B), U3.15 (3V3), U3.46 (3V3), U3.50 (3.3V)
- net +5V: now also JP1.1 (A), C26.2, C28.2, U3.48 (VIN)
- net +5V_ISO: now also C27.2
- net Buzzer_Logic: now also U3.12 (10_CS_MQSR)
- net CAN1_RX: now also U3.45 (23_A9_CRX1_MCLK1)
- net CAN1_TX: now also U3.44 (22_A8_CTX1)
- net CAN2_RX: now also U3.2 (0_RX1_CRX2_CS1)
- net CAN2_TX: now also U3.3 (1_TX1_CTX2_MISO1); no longer JP1.1 (A), JP1.2 (C)
- net CAN3_RX: now also U3.22 (30_CRX3)
- net CAN3_TX: now also U3.23 (31_CTX3)
- net Curr_Sens_High_3v3: now also U3.36 (14_A0_TX3_SPDIF_OUT)
- net Curr_Sens_Low_3v3: now also U3.37 (15_A1_RX3_SPDIF_IN)
- net ERROR_LED: now also U3.25 (33_MCLK2)
- net GND: now also H1.1, H2.1, H3.1, H4.1, C25.1, C26.1, C28.1, U3.1 (GND), U3.34 (GND), U3.47 (GND), U3.51 (GND)
- net GND_ISO: now also C27.1
- net HEARTBEAT_LED: now also U3.6 (4_BCLK2)
- net HSD_FAULT_RESET: now also U3.28 (36_CS)
- net HSD_MULTISENSE_A: now also U3.33 (41_A17)
- net HSD_MULTISENSE_B: now also U3.32 (40_A16)
- net HSD_SEL_0_A: now also U3.24 (32_OUT1B)
- net HSD_SEL_0_B: now also U3.29 (37_CS)
- net HSD_SEL_1_A: now also U3.19 (27_A13_SCK1)
- net HSD_SEL_1_B: now also U3.30 (38_CS1_IN1)
- net HSD_SEn_A: now also U3.18 (26_A12_MOSI1)
- net HSD_SEn_B: now also U3.31 (39_MISO1_OUT1A)
- net I2C_SCL: now also U3.16 (24_A10_TX6_SCL2)
- net I2C_SDA: now also U3.17 (25_A11_RX6_SDA2)
- net Logic_IN_1: now also U3.38 (16_A2_RX4_SCL1)
- net Logic_IN_2: now also U3.39 (17_A3_TX4_SDA1)
- net Logic_IN_3: now also U3.40 (18_A4_SDA)
- net Logic_IN_4: now also U3.41 (19_A5_SCL)
- net OUT1_HSD_LOGIC: now also U3.13 (11_MOSI_CTX1)
- net OUT2_HSD_LOGIC: now also U3.14 (12_MISO_MQSL)
- net OUT3_HSD_LOGIC: now also U3.42 (20_A6_TX5_LRCLK1)
- net OUT4_HSD_LOGIC: now also U3.43 (21_A7_RX5_BCLK1)
- net OUT5_LSD_LOGIC: now also U3.4 (2_OUT2)
- net OUT6_LSD_LOGIC: now also U3.5 (3_LRCLK2)
- net OUT7_LSD_LOGIC: now also U3.7 (5_IN2)
- net OUT8_LSD_LOGIC: now also U3.8 (6_OUT1D)
- net RS-485_DIR: now also U3.11 (9_OUT1C)
- net RTC_BATT_+: now also U3.49 (V_BATT_RTC)
- net RX_2_logic: now also U3.20 (28_RX7)
- net SERIAL_RX: now also U3.9 (7_RX2_OUT1A)
- net SERIAL_TX: now also U3.10 (8_TX2_IN1)
- net TX_2_logic: now also U3.21 (29_TX7)
- net RS-485_Rx renamed RX_3_logic
- net RX_3_logic: now also U3.27 (35_TX8)
- net RS-485_Tx renamed TX_3_logic
- net TX_3_logic: now also U3.26 (34_RX8); no longer JP1.3 (B)
- new net Isolated_UART1/Logic VCC: JP1.2 (C)
- no-connect marks 54 -> 56
Other:
- note added: "TODO - All molex connector footprints appear wider spaced than JLC Models"
- note removed: "CAN2/RS-485 Switch"
- moved on the sheet: U1

Commit message: 'Fixed' Molex Footprints - 2x8 not genuine molex, 4.2 instead of 5.5 RS
Parts:
- J1, J2, J6, J7: LCSC C2845777 -> C240829
- J4: footprint Connector_Molex:Molex_Mini-Fit_Jr_5566-16A_2x08_P4.20mm_Vertical -> user:Clone-Molex_Mini-Fit_Jr_5566-16A_2x05_P4.20mm_Vertical; LCSC C2845783 -> C293504
Connections:
- no-connect marks 56 -> 6
Other:
- note added: "43mW expected extreme 48V Input - 500mW is overkill..."
- note added: "No footprint items to hold part numbers for Teensy Headers Mounting hole symbols as schematic placeholders"
- note removed: "No footprint items to hold part numbers for Teensy Headers"
- note removed: "TODO: Free up some serial pins do CAN3 and RS485 don't have to share"
- note removed: "TODO: Multisense signals need to go to Analogue INputs!"

Commit message: Schematic Net Colours
Connections:
- net +12V_Fused: now reaches C1.1, D1.1 (K), F1.2, L1.1
- net +12V_Filtered: now reaches C2.1, L1.2, Q2.1 (S), Q2.2 (S), Q2.3 (S)
- net 12V_INPUT renamed +12V_INPUT
Other:
- note added: "43mW expected extreme 48V Input - 500mW might be overkill..."
- note added: "MCU Control"
- note removed: "43mW expected extreme 48V Input - 500mW is overkill..."
- note removed: "TODO - All molex connector footprints appear wider spaced than JLC Models"
- note removed: "TODO - check U14 Footprint. JLC Render is tiny SSOP16"
