File: CAN_Transceiver.kicad_sch (KiCad schematic)
At the start: 8 parts, among them SW2 SW_DIP_x01, U5 TJA1051T/3/1J

Commit message: Added 5V protection capacitors, altered 5V_ISO Output Caps, Corrected RX<>TX for Serial3
Connections:
- net GND: now also U5.8 (Rs)
Changed lines of the file:
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@@
 		)
+	)
+	(junction
+		(at 105.41 104.14)
+		(diameter 0)
+		(color 0 0 0 0)
 	)
 	(wire
@@
 	(wire
 		(pts
+			(xy 92.71 95.25) (xy 88.9 95.25)
+		)
+		(stroke
+			(width 0)
+			(type default)
+		)
+	)
+	(wire
+		(pts
 			(xy 123.19 148.59) (xy 123.19 144.78)
 		)
@@
 	(wire
 		(pts
+			(xy 88.9 104.14) (xy 105.41 104.14)
+		)
+		(stroke
+			(width 0)
+			(type default)
+		)
+	)
+	(wire
+		(pts
 			(xy 210.82 72.39) (xy 213.36 72.39)
 		)
 		(stroke
+			(width 0)
+			(type default)
+		)
+	)
+	(wire
+		(pts
+			(xy 88.9 95.25) (xy 88.9 104.14)
+		)
+		(stroke

Commit message: V0.1 as Manufactured
Parts:
- R4, R5: value 330R -> 330
Changed lines of the file:
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@@
 			)
 		)
-		(property "Value" "330R"
+		(property "Value" "330"
 			(at 85.09 87.884 90)
 			(effects
@@
 			)
 		)
-		(property "Value" "330R"
+		(property "Value" "330"
 			(at 85.09 85.09 90)
 			(effects
