File: UART_Isolated_Interface.kicad_sch (KiCad schematic)
At the start: 8 parts, among them U6 ISO7331C

Commit message: Connectors, high side circuits added, layout progressed
Connections:
- net GND renamed ISO_GND
Changed lines of the file:
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@@
 		)
 	)
-	(hierarchical_label "GND"
+	(hierarchical_label "ISO_GND"
 		(shape input)
 		(at 133.35 86.36 0)
@@
 		)
 	)
-	(hierarchical_label "GND"
+	(hierarchical_label "ISO_GND"
 		(shape input)
 		(at 134.62 109.22 0)
@@
 		)
 	)
-	(hierarchical_label "GND"
+	(hierarchical_label "ISO_GND"
 		(shape input)
 		(at 171.45 99.06 0)

Commit message: Finalised RS485 Circuit, Layout improvemnts, mounting holes, silkscreen...
Other:
- company: (none) -> eChook
- title: (none) -> BMS Comms Master Board
Changed lines of the file:
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@@
 	(generator_version "9.0")
 	(paper "A4")
+	(title_block
+		(title "BMS Comms Master Board")
+		(date "2025-05-21")
+		(rev "0.1")
+		(company "eChook")
+	)
 	(rectangle
 		(start 81.28 71.12)

Commit message: Pinout Review Complete, Altenative option for ISO CAN IC added
Parts:
- U6: value ISO7331C -> TI ISO7221ADR
Changed lines of the file:
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@@
 			)
 		)
-		(property "Value" "ISO7331C"
+		(property "Value" "TI ISO7221ADR"
 			(at 118.11 78.74 0)
 			(effects
@@
 			)
 		)
-		(property "Datasheet" "http://www.ti.com/general/docs/lit/getliterature.tsp?genericPartNumber=iso7321c&fileType=pdf"
+		(property "Datasheet" "https://www.lcsc.com/datasheet/C28037.pdf"
 			(at 118.11 88.9 0)
 			(effects

Commit message: V0.1 as Manufactured
Parts:
- R6, R7, R8, R9: value 330R -> 330
Changed lines of the file:
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@@
 			)
 		)
-		(property "Value" "330R"
+		(property "Value" "330"
 			(at 104.14 91.44 90)
 			(effects
@@
 			)
 		)
-		(property "Value" "330R"
+		(property "Value" "330"
 			(at 104.14 94.234 90)
 			(effects
@@
 			)
 		)
-		(property "Value" "330R"
+		(property "Value" "330"
 			(at 132.08 91.44 90)
 			(effects
@@
 			)
 		)
-		(property "Value" "330R"
+		(property "Value" "330"
 			(at 132.08 94.234 90)
 			(effects
